Commit message: Lab2 Almost

File: install/my_robot_description/share/my_robot_description/urdf/my_robot_gazebo.urdf (robot description, URDF)
Before this commit: robot my_robot, 5 links, 5 joints
Links:
- removed link camera_link_optical
- added link left_camera_link, mass 0.01; collision box size=0.05 0.05 0.05; visual box size=0.05 0.05 0.05
- added link left_camera_link_optical, mass 0.001
- added link right_camera_link, mass 0.01; collision box size=0.05 0.05 0.05; visual box size=0.05 0.05 0.05
- added link right_camera_link_optical, mass 0.001
- link base_link: geometry collision box size=0.4 0.3 0.1; visual box size=0.4 0.3 0.1
Joints:
- removed joint camera_joint
- removed joint camera_optical_joint
- added joint left_camera_joint: type fixed, parent base_link, child left_camera_link, origin xyz=0.15 0.05 0.075 rpy=0 0 0
- added joint left_camera_optical_joint: type fixed, parent left_camera_link, child left_camera_link_optical, origin xyz=0 0 0 rpy=-1.5707 0 -1.5707
- added joint right_camera_joint: type fixed, parent base_link, child right_camera_link, origin xyz=0.15 -0.05 0.075 rpy=0 0 0
- added joint right_camera_optical_joint: type fixed, parent right_camera_link, child right_camera_link_optical, origin xyz=0 0 0 rpy=-1.5707 0 -1.5707
- joint left_wheel_joint: origin xyz=-0.05 0.17 0 rpy=1.5707 0 0 -> xyz=-0.15 0.17 0 rpy=1.5707 0 0
- joint right_wheel_joint: origin xyz=-0.05 -0.17 0 rpy=1.5707 0 0 -> xyz=-0.15 -0.17 0 rpy=1.5707 0 0

File: src/my_robot_description/urdf/my_robot_gazebo.urdf (robot description, URDF)
Before this commit: robot my_robot, 5 links, 5 joints
Links:
- removed link camera_link_optical
- added link left_camera_link, mass 0.01; collision box size=0.05 0.05 0.05; visual box size=0.05 0.05 0.05
- added link left_camera_link_optical, mass 0.001
- added link right_camera_link, mass 0.01; collision box size=0.05 0.05 0.05; visual box size=0.05 0.05 0.05
- added link right_camera_link_optical, mass 0.001
- link base_link: geometry collision box size=0.4 0.3 0.1; visual box size=0.4 0.3 0.1
Joints:
- removed joint camera_joint
- removed joint camera_optical_joint
- added joint left_camera_joint: type fixed, parent base_link, child left_camera_link, origin xyz=0.15 0.05 0.075 rpy=0 0 0
- added joint left_camera_optical_joint: type fixed, parent left_camera_link, child left_camera_link_optical, origin xyz=0 0 0 rpy=-1.5707 0 -1.5707
- added joint right_camera_joint: type fixed, parent base_link, child right_camera_link, origin xyz=0.15 -0.05 0.075 rpy=0 0 0
- added joint right_camera_optical_joint: type fixed, parent right_camera_link, child right_camera_link_optical, origin xyz=0 0 0 rpy=-1.5707 0 -1.5707
- joint left_wheel_joint: origin xyz=-0.05 0.17 0 rpy=1.5707 0 0 -> xyz=-0.15 0.17 0 rpy=1.5707 0 0
- joint right_wheel_joint: origin xyz=-0.05 -0.17 0 rpy=1.5707 0 0 -> xyz=-0.15 -0.17 0 rpy=1.5707 0 0
