Commit message: Update Lab2 Robot

File: install/my_robot_description/share/my_robot_description/urdf/my_robot.urdf (robot description, URDF)
Before this commit: robot my_robot, 8 links, 7 joints
Links:
- added link top_link, mass 1.0; collision cylinder length=0.07 radius=0.1; visual cylinder length=0.07 radius=0.1
- link base_link: geometry collision box size=0.4 0.3 0.1; visual box size=0.4 0.3 0.1
Joints:
- added joint top_link_joint: type fixed, parent base_link, child top_link, origin xyz=0 0 0.085 rpy=0 0 0
- joint left_wheel_joint: origin xyz=-0.15 0.7 0 rpy=1.5707 0 0 -> xyz=-0.15 0.17 0 rpy=1.5707 0 0
- joint right_wheel_joint: origin xyz=-0.15 -0.7 0 rpy=1.5707 0 0 -> xyz=-0.15 -0.17 0 rpy=1.5707 0 0

File: install/my_robot_description/share/my_robot_description/urdf/my_robot_gazebo.urdf (robot description, URDF)
Before this commit: robot my_robot, 8 links, 7 joints
Links:
- added link top_link, mass 1.0; collision cylinder length=0.07 radius=0.1; visual cylinder length=0.07 radius=0.1
Joints:
- added joint top_link_joint: type fixed, parent base_link, child top_link, origin xyz=0 0 0.085 rpy=0 0 0
